Commit message: update urdf files

File: models/block/model0.urdf (robot description, URDF)
Before this commit: robot block, 1 links, 0 joints
Links:
- link block: mass 4.98952 -> 2.49476

File: models/block/model1.urdf (robot description, URDF)
Before this commit: robot block, 1 links, 0 joints
Links:
- link block: mass 3.62874 -> 1.81437

File: models/block/model2.urdf (robot description, URDF)
Before this commit: robot block, 1 links, 0 joints
Links:
- link block: mass 2.26796 -> 1.13398

File: models/block/model3.urdf (robot description, URDF)
Before this commit: robot block, 1 links, 0 joints
Links:
- link block: mass 1.36078 -> 0.68039

File: models/block/model4.urdf (robot description, URDF)
Before this commit: robot block, 1 links, 0 joints
Links:
- link block: mass 0.453592 -> 0.226796

Commit message: new change

File: models/block/model0.urdf (robot description, URDF)
Before this commit: robot block, 1 links, 0 joints
Links:
- link block: geometry collision box size=0.045 0.045 0.045; visual box size=0.045 0.045 0.045

File: models/block/model1.urdf (robot description, URDF)
Before this commit: robot block, 1 links, 0 joints
Links:
- link block: geometry collision box size=0.045 0.045 0.045; visual box size=0.045 0.045 0.045

File: models/block/model2.urdf (robot description, URDF)
Before this commit: robot block, 1 links, 0 joints
Links:
- link block: geometry collision box size=0.045 0.045 0.045; visual box size=0.045 0.045 0.045

File: models/block/model3.urdf (robot description, URDF)
Before this commit: robot block, 1 links, 0 joints
Links:
- link block: geometry collision box size=0.045 0.045 0.045; visual box size=0.045 0.045 0.045

File: models/block/model4.urdf (robot description, URDF)
Before this commit: robot block, 1 links, 0 joints
Links:
- link block: geometry collision box size=0.045 0.045 0.045; visual box size=0.045 0.045 0.045

Commit message: added noise and seperated task to pick,grasp and place

File: models/block/model0.urdf (robot description, URDF)
Before this commit: robot block, 1 links, 0 joints
Links:
- link block: mass 2.49476 -> 5

File: models/block/model1.urdf (robot description, URDF)
Before this commit: robot block, 1 links, 0 joints
Links:
- link block: mass 1.81437 -> 4.5

File: models/block/model2.urdf (robot description, URDF)
Before this commit: robot block, 1 links, 0 joints
Links:
- link block: mass 1.13398 -> 4

File: models/block/model3.urdf (robot description, URDF)
Before this commit: robot block, 1 links, 0 joints
Links:
- link block: mass 0.68039 -> 3.5

File: models/block/model4.urdf (robot description, URDF)
Before this commit: robot block, 1 links, 0 joints
Links:
- link block: mass 0.226796 -> 3
